File: kicad/panel.kicad_pcb (KiCad board)
At the start: 4 copper layers, 273 x 119.9 mm, 234 parts, among them Q1 PMF170XP,115, Q2 FS8205A_C2830320, SW1 TS-1088-AR02016, U1 SN74LVC1G17DBVR, U10 SN74LVC1G74DQER, U2 E73-2G4M08S1C, U3 SN74LVC1G74DQER, U4 S2B-PH-K-S(LF)(SN), U5 BL8573CS8TR, U6 DW01A_C42380662, U7 LP5024RSMR, U8 MAX17048, U9 USBLC6-2SC6, X1 FC-13532.768KHZ9PF20PPM

Commit message: rewired and finalized right side. updated panel. changed dnp of some components on both sides
Parts:
- removed the BAT+ at (269.7, 33.1)
- removed the BAT+ at (60.3, 44.4)
- removed the C1 at (64.7, 94.0)
- removed the C1 at (280.2, 73.2)
- removed the C3 at (280.2, 75.2)
- removed the C3 at (64.7, 92.0)
- removed the C5 at (57.0, 79.6)
- removed the C5 at (288.3, 87.3)
- removed the C6 at (295.4, 93.2)
- removed the C6 at (59.3, 79.6)
- removed the C7 at (278.1, 75.1)
- removed the C7 at (66.9, 92.0)
- removed the C8 at (69.0, 85.1)
- removed the C8 at (278.1, 81.4)
- removed the C9 at (280.5, 64.0)
- removed the C9 at (63.9, 64.9)
- removed the D1 at (62.2, 62.7)
- removed the D1 at (274.8, 57.9)
- removed the D10 at (124.3, 67.4)
- removed the D10 at (221.4, 56.7)
- removed the D11 at (227.7, 74.1)
- removed the D11 at (122.3, 67.4)
- removed the D12 at (264.9, 117.1)
- removed the D12 at (85.1, 110.4)
- removed the D13 at (240.0, 45.9)
- removed the D13 at (105.7, 56.6)
- removed the D14 at (105.7, 78.1)
- removed the D14 at (240.0, 67.4)
- removed the D15 at (103.7, 99.6)
- removed the D15 at (240.0, 88.9)
- removed the D16 at (283.5, 106.4)
- removed the D16 at (79.7, 110.3)
- removed the D17 at (258.6, 56.7)
- removed the D17 at (87.1, 67.4)
- removed the D18 at (87.1, 88.9)
- removed the D18 at (258.6, 78.2)
- removed the D19 at (258.6, 99.7)
- removed the D19 at (98.6, 99.5)
- removed the D2 at (184.2, 56.7)
- removed the D2 at (160.2, 67.3)
- removed the D20 at (302.2, 117.1)
- removed the D20 at (55.3, 110.3)
- removed the D3 at (184.2, 78.2)
- removed the D3 at (165.0, 88.8)
- removed the D4 at (159.9, 88.7)
- removed the D4 at (190.4, 95.6)
- removed the D5 at (143.0, 56.6)
- removed the D5 at (202.8, 45.9)
- removed the D6 at (202.8, 67.4)
- removed the D6 at (143.6, 78.0)
- removed the D7 at (141.5, 78.1)
- removed the D7 at (209.1, 84.9)
- removed the D8 at (246.3, 106.4)
- removed the D8 at (105.7, 99.6)
- removed the D9 at (124.3, 45.9)
- removed the D9 at (221.4, 35.2)
- removed the F1 at (281.7, 35.4)
- removed the F1 at (71.3, 47.0)
- removed the G** at (278.5, 65.4)
- removed the G** at (57.1, 76.0)
- removed the GND at (267.8, 36.5)
- removed the GND at (57.2, 47.2)
- removed the H1 at (44.3, 73.2)
- removed the H1 at (300.9, 61.6)
- removed the L1 at (282.7, 84.7)
- removed the L1 at (62.6, 82.9)
- removed the LED1 at (158.3, 52.5)
- removed the LED1 at (186.6, 41.8)
- removed the LED10 at (121.1, 73.9)
- removed the LED10 at (223.8, 63.3)
- removed the LED11 at (261.1, 106.3)
- removed the LED11 at (83.8, 117.0)
- removed the LED12 at (102.5, 41.7)
- removed the LED12 at (242.4, 31.0)
- removed the LED13 at (242.4, 52.5)
- removed the LED13 at (102.5, 63.2)
- removed the LED14 at (102.5, 84.7)
- removed the LED14 at (242.4, 74.0)
- removed the LED15 at (279.8, 95.6)
- removed the LED15 at (65.1, 106.3)
- removed the LED16 at (261.1, 41.8)
- removed the LED16 at (83.8, 52.5)
- removed the LED17 at (83.8, 74.0)
- removed the LED17 at (261.1, 63.3)
- removed the LED18 at (261.1, 84.8)
- removed the LED18 at (83.8, 95.5)
- removed the LED19 at (46.6, 117.0)
- removed the LED19 at (298.3, 106.3)
- removed the LED2 at (186.6, 63.3)
- removed the LED2 at (158.3, 74.0)
- removed the LED20 at (298.3, 41.8)
- removed the LED20 at (46.6, 52.5)
- removed the LED3 at (186.6, 84.8)
- removed the LED3 at (158.3, 95.5)
- removed the LED4 at (205.2, 31.0)
- removed the LED4 at (139.7, 41.7)
- removed the LED5 at (205.2, 52.5)
- removed the LED5 at (139.7, 63.2)
- removed the LED6 at (205.2, 74.0)
- removed the LED6 at (139.7, 84.7)
- removed the LED7 at (102.4, 106.2)
- removed the LED7 at (242.5, 95.6)
- removed the LED8 at (121.1, 30.9)
- removed the LED8 at (223.8, 20.3)
- removed the LED9 at (121.1, 52.5)
- removed the LED9 at (223.8, 41.8)
- removed the PWR at (270.4, 51.2)
- removed the PWR at (69.8, 74.1)
- removed the Q1 at (278.0, 52.6)
- removed the Q1 at (69.5, 67.9)
- removed the Q2 at (280.9, 45.5)
- removed the Q2 at (70.3, 57.1)
- removed the R1 at (294.6, 69.3)
- removed the R1 at (57.5, 65.3)
- removed the R10 at (66.2, 45.8)
- removed the R10 at (276.7, 34.1)
- removed the R11 at (281.5, 40.7)
- removed the R11 at (70.7, 52.1)
- removed the R13 at (68.5, 80.7)
- removed the R13 at (272.2, 39.8)
- removed the R14 at (278.1, 80.2)
- removed the R14 at (67.4, 87.8)
- removed the R16 at (66.3, 87.8)
- removed the R16 at (278.1, 79.0)
- removed the R17 at (66.9, 89.5)
- removed the R17 at (278.1, 77.7)
- removed the R2 at (293.4, 69.3)
- removed the R2 at (57.5, 67.5)
- removed the R5 at (280.8, 56.4)
- removed the R5 at (62.2, 61.4)
- removed the R6 at (66.9, 90.8)
- removed the R6 at (278.1, 76.4)
- removed the R7 at (273.2, 53.3)
- removed the R7 at (62.2, 63.9)
- removed the R8 at (65.4, 82.3)
- removed the R8 at (292.9, 93.2)
- removed the R9 at (278.0, 34.1)
- removed the R9 at (68.8, 45.8)
- removed the REF** at (233.9, 45.9)
- removed the REF** at (92.3, 110.3)
- removed the REF** at (148.2, 78.0)
- removed the REF** at (252.5, 99.6)
- removed the REF** at (111.0, 56.5)
- removed the REF** at (196.7, 67.4)
- removed the S1 at (184.3, 45.9)
- removed the S1 at (160.6, 56.5)
- removed the S10 at (221.5, 67.4)
- removed the S10 at (123.4, 78.0)
- removed the S11 at (258.7, 110.4)
- removed the S11 at (86.2, 121.0)
- removed the S12 at (240.1, 35.1)
- removed the S12 at (104.8, 45.8)
- removed the S13 at (240.1, 56.6)
- removed the S13 at (104.8, 67.3)
- removed the S14 at (240.1, 78.1)
- removed the S14 at (104.8, 88.8)
- removed the S15 at (277.4, 99.6)
- removed the S15 at (67.5, 110.3)
- removed the S16 at (258.7, 45.9)
- removed the S16 at (86.2, 56.5)
- removed the S17 at (258.7, 67.4)
- removed the S17 at (86.2, 78.0)
- removed the S18 at (258.7, 88.9)
- removed the S18 at (86.2, 99.5)
- removed the S19 at (296.0, 110.4)
- removed the S19 at (48.9, 121.0)
- removed the S2 at (184.3, 67.4)
- removed the S2 at (160.6, 78.0)
- removed the S20 at (296.0, 45.9)
- removed the S20 at (48.9, 56.5)
- removed the S3 at (184.3, 88.9)
- removed the S3 at (160.6, 99.5)
- removed the S4 at (202.9, 35.1)
- removed the S4 at (142.0, 45.8)
- removed the S5 at (202.9, 56.6)
- removed the S5 at (142.0, 67.3)
- removed the S6 at (202.9, 78.1)
- removed the S6 at (142.0, 88.8)
- removed the S7 at (240.1, 99.6)
- removed the S7 at (104.8, 110.3)
- removed the S8 at (221.5, 24.4)
- removed the S8 at (123.4, 35.0)
- removed the S9 at (221.5, 45.9)
- removed the S9 at (123.4, 56.5)
- removed the SW1 at (63.4, 79.4)
- removed the SW1 at (294.0, 91.0)
- removed the U1 at (278.1, 56.8)
- removed the U1 at (66.2, 66.6)
- removed the U2 at (291.4, 78.1)
- removed the U2 at (53.5, 88.8)
- removed the U4 at (61.6, 47.4)
- removed the U4 at (272.0, 35.9)
- removed the U5 at (277.0, 40.5)
- removed the U5 at (66.6, 52.1)
- removed the U6 at (276.2, 45.5)
- removed the U6 at (65.8, 57.1)
- removed the U7 at (71.2, 88.9)
- removed the U7 at (273.7, 78.3)
- removed the U8 at (280.1, 66.3)
- removed the U8 at (69.9, 82.6)
- removed the U9 at (285.1, 32.0)
- removed the U9 at (75.1, 42.7)
- removed the USBC1 at (277.4, 28.7)
- removed the USBC1 at (67.5, 39.4)
- removed the VBUS at (286.5, 37.0)
- removed the VBUS at (76.0, 48.9)
- removed the VDD_nrf at (278.6, 61.9)
- removed the VDD_nrf at (58.6, 75.8)
- removed the X1 at (62.8, 92.9)
- removed the X1 at (282.1, 74.3)
- added BAT+: TestPoint_THTPad_D2.0mm_Drill1.0mm, TestPoint:TestPoint_THTPad_D2.0mm_Drill1.0mm, F.Cu at (60.9, 43.9)
- added BAT+: TestPoint_THTPad_D2.0mm_Drill1.0mm, TestPoint:TestPoint_THTPad_D2.0mm_Drill1.0mm, F.Cu at (269.7, 33.1)
- added C1: 0402CG120J500NT, easyeda2kicad:C0402, F.Cu at (280.2, 73.2)
- added C1: 0402CG120J500NT, easyeda2kicad:C0402, F.Cu at (64.7, 94.0)
- added C3: 0402CG120J500NT, easyeda2kicad:C0402, F.Cu at (280.2, 75.2)
- added C3: 0402CG120J500NT, easyeda2kicad:C0402, F.Cu at (64.7, 92.0)
- added C5: ZRB15XR61A475KE01D, easyeda2kicad:C0402, F.Cu at (288.3, 87.3)
- added C5: ZRB15XR61A475KE01D, easyeda2kicad:C0402, F.Cu at (57.1, 79.4)
- added C6: CL05B104KB54PNC, easyeda2kicad:C0402, F.Cu at (60.4, 77.2)
- added C6: CL05B104KB54PNC, easyeda2kicad:C0402, F.Cu at (295.4, 93.2)
- added C7: CL05A105KA5NQNC, easyeda2kicad:C0402, F.Cu at (66.9, 92.0)
- added C7: CL05A105KA5NQNC, easyeda2kicad:C0402, F.Cu at (278.1, 75.1)
- added C8: CL05A105KA5NQNC, easyeda2kicad:C0402, F.Cu at (66.9, 85.7)
- added C8: CL05A105KA5NQNC, easyeda2kicad:C0402, F.Cu at (278.1, 81.4)
- added C9: CL05B104KB54PNC, easyeda2kicad:C0402, F.Cu at (280.5, 64.1)
- added C9: CL05A105KA5NQNC, easyeda2kicad:C0402, F.Cu at (71.0, 70.8)
- added D1: NSR05F20NXT5G, easyeda2kicad:DSN2_L1.0-W0.6-RD, F.Cu at (68.6, 70.7)
- added D1: NSR05F20NXT5G, easyeda2kicad:DSN2_L1.0-W0.6-RD, F.Cu at (274.8, 57.9)
- added D10: CDSQC4148-HF, easyeda2kicad:X1-DFN1006-2_L1.0-W0.6-RD, F.Cu at (221.4, 56.7)
- added D10: CDSQC4148-HF, easyeda2kicad:X1-DFN1006-2_L1.0-W0.6-RD, F.Cu at (123.4, 45.7)
- added D11: CDSQC4148-HF, easyeda2kicad:X1-DFN1006-2_L1.0-W0.6-RD, F.Cu at (123.4, 67.1)
- added D11: CDSQC4148-HF, easyeda2kicad:X1-DFN1006-2_L1.0-W0.6-RD, F.Cu at (227.7, 74.1)
- added D12: CDSQC4148-HF, easyeda2kicad:X1-DFN1006-2_L1.0-W0.6-RD, F.Cu at (96.9, 120.7)
- added D12: CDSQC4148-HF, easyeda2kicad:X1-DFN1006-2_L1.0-W0.6-RD, F.Cu at (264.9, 117.1)
- added D13: CDSQC4148-HF, easyeda2kicad:X1-DFN1006-2_L1.0-W0.6-RD, F.Cu at (240.0, 46.0)
- added D13: CDSQC4148-HF, easyeda2kicad:X1-DFN1006-2_L1.0-W0.6-RD, F.Cu at (107.8, 56.4)
- added D14: CDSQC4148-HF, easyeda2kicad:X1-DFN1006-2_L1.0-W0.6-RD, F.Cu at (104.8, 56.3)
- added D14: CDSQC4148-HF, easyeda2kicad:X1-DFN1006-2_L1.0-W0.6-RD, F.Cu at (240.0, 67.5)
- added D15: CDSQC4148-HF, easyeda2kicad:X1-DFN1006-2_L1.0-W0.6-RD, F.Cu at (104.8, 77.8)
- added D15: CDSQC4148-HF, easyeda2kicad:X1-DFN1006-2_L1.0-W0.6-RD, F.Cu at (240.0, 89.0)
- added D16: CDSQC4148-HF, easyeda2kicad:X1-DFN1006-2_L1.0-W0.6-RD, F.Cu at (283.5, 106.4)
- added D16: CDSQC4148-HF, easyeda2kicad:X1-DFN1006-2_L1.0-W0.6-RD, F.Cu at (72.9, 119.2)
- added D17: CDSQC4148-HF, easyeda2kicad:X1-DFN1006-2_L1.0-W0.6-RD, F.Cu at (89.2, 67.2)
- added D17: CDSQC4148-HF, easyeda2kicad:X1-DFN1006-2_L1.0-W0.6-RD, F.Cu at (258.6, 56.7)
- added D18: CDSQC4148-HF, easyeda2kicad:X1-DFN1006-2_L1.0-W0.6-RD, F.Cu at (258.6, 78.2)
- added D18: CDSQC4148-HF, easyeda2kicad:X1-DFN1006-2_L1.0-W0.6-RD, F.Cu at (86.2, 67.1)
- added D19: CDSQC4148-HF, easyeda2kicad:X1-DFN1006-2_L1.0-W0.6-RD, F.Cu at (258.6, 99.7)
- added D19: CDSQC4148-HF, easyeda2kicad:X1-DFN1006-2_L1.0-W0.6-RD, F.Cu at (86.2, 88.7)
- added D2: CDSQC4148-HF, easyeda2kicad:X1-DFN1006-2_L1.0-W0.6-RD, F.Cu at (163.6, 67.2)
- added D2: CDSQC4148-HF, easyeda2kicad:X1-DFN1006-2_L1.0-W0.6-RD, F.Cu at (184.2, 56.7)
- added D20: CDSQC4148-HF, easyeda2kicad:X1-DFN1006-2_L1.0-W0.6-RD, F.Cu at (302.2, 117.1)
- added D20: CDSQC4148-HF, easyeda2kicad:X1-DFN1006-2_L1.0-W0.6-RD, F.Cu at (59.6, 120.7)
- added D3: CDSQC4148-HF, easyeda2kicad:X1-DFN1006-2_L1.0-W0.6-RD, F.Cu at (160.6, 67.1)
- added D3: CDSQC4148-HF, easyeda2kicad:X1-DFN1006-2_L1.0-W0.6-RD, F.Cu at (184.2, 78.2)
- added D4: CDSQC4148-HF, easyeda2kicad:X1-DFN1006-2_L1.0-W0.6-RD, F.Cu at (190.4, 95.6)
- added D4: CDSQC4148-HF, easyeda2kicad:X1-DFN1006-2_L1.0-W0.6-RD, F.Cu at (160.6, 88.7)
- added D5: CDSQC4148-HF, easyeda2kicad:X1-DFN1006-2_L1.0-W0.6-RD, F.Cu at (202.8, 46.0)
- added D5: CDSQC4148-HF, easyeda2kicad:X1-DFN1006-2_L1.0-W0.6-RD, F.Cu at (145.0, 56.4)
- added D6: CDSQC4148-HF, easyeda2kicad:X1-DFN1006-2_L1.0-W0.6-RD, F.Cu at (142.0, 56.3)
- added D6: CDSQC4148-HF, easyeda2kicad:X1-DFN1006-2_L1.0-W0.6-RD, F.Cu at (202.8, 67.5)
- added D7: CDSQC4148-HF, easyeda2kicad:X1-DFN1006-2_L1.0-W0.6-RD, F.Cu at (209.1, 84.9)
- added D7: CDSQC4148-HF, easyeda2kicad:X1-DFN1006-2_L1.0-W0.6-RD, F.Cu at (142.0, 78.0)
- added D8: CDSQC4148-HF, easyeda2kicad:X1-DFN1006-2_L1.0-W0.6-RD, F.Cu at (246.3, 106.4)
- added D8: CDSQC4148-HF, easyeda2kicad:X1-DFN1006-2_L1.0-W0.6-RD, F.Cu at (115.5, 109.9)
- added D9: CDSQC4148-HF, easyeda2kicad:X1-DFN1006-2_L1.0-W0.6-RD, F.Cu at (221.4, 35.2)
- added D9: CDSQC4148-HF, easyeda2kicad:X1-DFN1006-2_L1.0-W0.6-RD, F.Cu at (126.4, 45.7)
- added F1: SMD1206-150C-16V, easyeda2kicad:F1206, F.Cu at (281.7, 35.4)
- added F1: SMD1206-150C-16V, easyeda2kicad:F1206, F.Cu at (69.1, 46.8)
- added G**: LOGO, images:handy, B.Cu at (278.5, 65.4)
- added G**: LOGO, images:handy, B.Cu at (57.1, 76.0)
- added GND: TestPoint_THTPad_D2.0mm_Drill1.0mm, TestPoint:TestPoint_THTPad_D2.0mm_Drill1.0mm, F.Cu at (57.7, 47.0)
- added GND: TestPoint_THTPad_D2.0mm_Drill1.0mm, TestPoint:TestPoint_THTPad_D2.0mm_Drill1.0mm, F.Cu at (267.8, 36.5)
- added H1: HC-PM254-8.5H-1X3PW, easyeda2kicad:HDR-TH_3P-P2.54_HC-PM254-8.5H-1X3PW, F.Cu at (300.9, 61.6)
- added H1: HC-PM254-8.5H-1X3PW, easyeda2kicad:HDR-TH_3P-P2.54_HC-PM254-8.5H-1X3PW, F.Cu at (43.8, 72.6)
- added L1: BRC2016T100K, easyeda2kicad:IND-SMD_L2.0-W1.6_BRC2016, F.Cu at (63.6, 82.7)
- added L1: BRC2016T100K, easyeda2kicad:IND-SMD_L2.0-W1.6_BRC2016, F.Cu at (282.7, 84.7)
- added LED1: OSO5PAS1C1A-1MA, easyeda2kicad:LED-SMD_L3.2-W2.8-LS3.5-RD-BLUE, F.Cu at (186.6, 41.8)
- added LED1: OSO5PAS1C1A-1MA, easyeda2kicad:LED-SMD_L3.2-W2.8-LS3.5-RD-BLUE, F.Cu at (158.3, 52.5)
- added LED10: OSO5PAS1C1A-1MA, easyeda2kicad:LED-SMD_L3.2-W2.8-LS3.5-RD-BLUE, F.Cu at (223.8, 63.3)
- added LED10: OSO5PAS1C1A-1MA, easyeda2kicad:LED-SMD_L3.2-W2.8-LS3.5-RD-BLUE, F.Cu at (121.1, 73.9)
- added LED11: OSO5PAS1C1A-1MA, easyeda2kicad:LED-SMD_L3.2-W2.8-LS3.5-RD-BLUE, F.Cu at (261.1, 106.3)
- added LED11: OSO5PAS1C1A-1MA, easyeda2kicad:LED-SMD_L3.2-W2.8-LS3.5-RD-BLUE, F.Cu at (83.8, 117.0)
- added LED12: OSO5PAS1C1A-1MA, easyeda2kicad:LED-SMD_L3.2-W2.8-LS3.5-RD-BLUE, F.Cu at (242.4, 31.0)
- added LED12: OSO5PAS1C1A-1MA, easyeda2kicad:LED-SMD_L3.2-W2.8-LS3.5-RD-BLUE, F.Cu at (102.5, 41.7)
- added LED13: OSO5PAS1C1A-1MA, easyeda2kicad:LED-SMD_L3.2-W2.8-LS3.5-RD-BLUE, F.Cu at (242.4, 52.5)
- added LED13: OSO5PAS1C1A-1MA, easyeda2kicad:LED-SMD_L3.2-W2.8-LS3.5-RD-BLUE, F.Cu at (102.5, 63.2)
- added LED14: OSO5PAS1C1A-1MA, easyeda2kicad:LED-SMD_L3.2-W2.8-LS3.5-RD-BLUE, F.Cu at (242.4, 74.0)
- added LED14: OSO5PAS1C1A-1MA, easyeda2kicad:LED-SMD_L3.2-W2.8-LS3.5-RD-BLUE, F.Cu at (102.5, 84.7)
- added LED15: OSO5PAS1C1A-1MA, easyeda2kicad:LED-SMD_L3.2-W2.8-LS3.5-RD-BLUE, F.Cu at (279.8, 95.6)
- added LED15: OSO5PAS1C1A-1MA, easyeda2kicad:LED-SMD_L3.2-W2.8-LS3.5-RD-BLUE, F.Cu at (65.1, 106.3)
- added LED16: OSO5PAS1C1A-1MA, easyeda2kicad:LED-SMD_L3.2-W2.8-LS3.5-RD-BLUE, F.Cu at (83.8, 52.5)
- added LED16: OSO5PAS1C1A-1MA, easyeda2kicad:LED-SMD_L3.2-W2.8-LS3.5-RD-BLUE, F.Cu at (261.1, 41.8)
- added LED17: OSO5PAS1C1A-1MA, easyeda2kicad:LED-SMD_L3.2-W2.8-LS3.5-RD-BLUE, F.Cu at (83.8, 74.0)
- added LED17: OSO5PAS1C1A-1MA, easyeda2kicad:LED-SMD_L3.2-W2.8-LS3.5-RD-BLUE, F.Cu at (261.1, 63.3)
- added LED18: OSO5PAS1C1A-1MA, easyeda2kicad:LED-SMD_L3.2-W2.8-LS3.5-RD-BLUE, F.Cu at (83.8, 95.5)
- added LED18: OSO5PAS1C1A-1MA, easyeda2kicad:LED-SMD_L3.2-W2.8-LS3.5-RD-BLUE, F.Cu at (261.1, 84.8)
- added LED19: OSO5PAS1C1A-1MA, easyeda2kicad:LED-SMD_L3.2-W2.8-LS3.5-RD-BLUE, F.Cu at (298.3, 106.3)
- added LED19: OSO5PAS1C1A-1MA, easyeda2kicad:LED-SMD_L3.2-W2.8-LS3.5-RD-BLUE, F.Cu at (46.6, 117.0)
- added LED2: OSO5PAS1C1A-1MA, easyeda2kicad:LED-SMD_L3.2-W2.8-LS3.5-RD-BLUE, F.Cu at (158.3, 74.0)
- added LED2: OSO5PAS1C1A-1MA, easyeda2kicad:LED-SMD_L3.2-W2.8-LS3.5-RD-BLUE, F.Cu at (186.6, 63.3)
- added LED20: OSO5PAS1C1A-1MA, easyeda2kicad:LED-SMD_L3.2-W2.8-LS3.5-RD-BLUE, F.Cu at (298.3, 41.8)
- added LED20: OSO5PAS1C1A-1MA, easyeda2kicad:LED-SMD_L3.2-W2.8-LS3.5-RD-BLUE, F.Cu at (46.6, 52.5)
- added LED3: OSO5PAS1C1A-1MA, easyeda2kicad:LED-SMD_L3.2-W2.8-LS3.5-RD-BLUE, F.Cu at (158.3, 95.5)
- added LED3: OSO5PAS1C1A-1MA, easyeda2kicad:LED-SMD_L3.2-W2.8-LS3.5-RD-BLUE, F.Cu at (186.6, 84.8)
- added LED4: OSO5PAS1C1A-1MA, easyeda2kicad:LED-SMD_L3.2-W2.8-LS3.5-RD-BLUE, F.Cu at (205.2, 31.0)
- added LED4: OSO5PAS1C1A-1MA, easyeda2kicad:LED-SMD_L3.2-W2.8-LS3.5-RD-BLUE, F.Cu at (139.7, 41.7)
- added LED5: OSO5PAS1C1A-1MA, easyeda2kicad:LED-SMD_L3.2-W2.8-LS3.5-RD-BLUE, F.Cu at (205.2, 52.5)
- added LED5: OSO5PAS1C1A-1MA, easyeda2kicad:LED-SMD_L3.2-W2.8-LS3.5-RD-BLUE, F.Cu at (139.7, 63.2)
- added LED6: OSO5PAS1C1A-1MA, easyeda2kicad:LED-SMD_L3.2-W2.8-LS3.5-RD-BLUE, F.Cu at (205.2, 74.0)
- added LED6: OSO5PAS1C1A-1MA, easyeda2kicad:LED-SMD_L3.2-W2.8-LS3.5-RD-BLUE, F.Cu at (139.7, 84.7)
- added LED7: OSO5PAS1C1A-1MA, easyeda2kicad:LED-SMD_L3.2-W2.8-LS3.5-RD-BLUE, F.Cu at (102.4, 106.2)
- added LED7: OSO5PAS1C1A-1MA, easyeda2kicad:LED-SMD_L3.2-W2.8-LS3.5-RD-BLUE, F.Cu at (242.5, 95.6)
- added LED8: OSO5PAS1C1A-1MA, easyeda2kicad:LED-SMD_L3.2-W2.8-LS3.5-RD-BLUE, F.Cu at (223.8, 20.3)
- added LED8: OSO5PAS1C1A-1MA, easyeda2kicad:LED-SMD_L3.2-W2.8-LS3.5-RD-BLUE, F.Cu at (121.1, 30.9)
- added LED9: OSO5PAS1C1A-1MA, easyeda2kicad:LED-SMD_L3.2-W2.8-LS3.5-RD-BLUE, F.Cu at (121.1, 52.5)
- added LED9: OSO5PAS1C1A-1MA, easyeda2kicad:LED-SMD_L3.2-W2.8-LS3.5-RD-BLUE, F.Cu at (223.8, 41.8)
- added PWR: TestPoint_THTPad_D2.0mm_Drill1.0mm, TestPoint:TestPoint_THTPad_D2.0mm_Drill1.0mm, F.Cu at (270.4, 51.2)
- added PWR: TestPoint_THTPad_D2.0mm_Drill1.0mm, TestPoint:TestPoint_THTPad_D2.0mm_Drill1.0mm, F.Cu at (75.1, 66.8)
- added Q1: PMF170XP,115, easyeda2kicad:SOT-323-3_L2.0-W1.3-P1.30-LS2.1-BR, F.Cu at (278.0, 52.6)
- added Q1: PMF170XP,115, easyeda2kicad:SOT-323-3_L2.0-W1.3-P1.30-LS2.1-BR, F.Cu at (72.6, 61.8)
- added Q2: FS8205A_C2830320, easyeda2kicad:SOT-23-6_L2.9-W1.6-P0.95-LS2.8-BR, F.Cu at (70.4, 56.3)
- added Q2: FS8205A_C2830320, easyeda2kicad:SOT-23-6_L2.9-W1.6-P0.95-LS2.8-BR, F.Cu at (280.9, 45.5)
- added R1: 0402WGF1004TCE, easyeda2kicad:R0402, F.Cu at (294.6, 69.4)
- added R1: 0402WGF1004TCE, easyeda2kicad:R0402, F.Cu at (53.0, 67.7)
- added R10: 0402WGF5101TCE, easyeda2kicad:R0402, F.Cu at (276.0, 34.7)
- added R10: 0402WGF5101TCE, easyeda2kicad:R0402, F.Cu at (66.6, 44.7)
- added R11: RC0402FR-07680RL, easyeda2kicad:R0402, F.Cu at (281.5, 40.7)
- added R11: RC0402FR-07680RL, easyeda2kicad:R0402, F.Cu at (72.2, 50.9)
- added R13: 0402WGF1002TCE, easyeda2kicad:R0402, F.Cu at (272.2, 39.9)
- added R13: 0402WGF1002TCE, easyeda2kicad:R0402, F.Cu at (60.6, 68.1)
- added R14: 0402WGF5101TCE, easyeda2kicad:R0402, F.Cu at (66.9, 87.0)
- added R14: 0402WGF5101TCE, easyeda2kicad:R0402, F.Cu at (278.1, 80.2)
- added R16: 0402WGF5101TCE, easyeda2kicad:R0402, F.Cu at (66.9, 88.3)
- added R16: 0402WGF5101TCE, easyeda2kicad:R0402, F.Cu at (278.1, 79.0)
- added R17: 0402WGF1004TCE, easyeda2kicad:R0402, F.Cu at (66.9, 89.5)
- added R17: 0402WGF1004TCE, easyeda2kicad:R0402, F.Cu at (278.1, 77.7)
- added R2: WR04W2494FTL, easyeda2kicad:R0402, F.Cu at (293.4, 69.4)
- added R2: WR04W2494FTL, easyeda2kicad:R0402, F.Cu at (50.2, 67.7)
- added R5: RTT022614FTH, easyeda2kicad:R0402, F.Cu at (280.8, 56.5)
- added R5: 0402WGF1002TCE, easyeda2kicad:R0402, F.Cu at (67.3, 70.8)
- added R6: ERA2AED753X, easyeda2kicad:R0402, F.Cu at (278.1, 76.4)
- added R6: ERA2AED753X, easyeda2kicad:R0402, F.Cu at (66.9, 90.8)
- added R7: 0402WGF1002TCE, easyeda2kicad:R0402, F.Cu at (273.2, 53.3)
- added R7: RTT022614FTH, easyeda2kicad:R0402, F.Cu at (69.8, 70.8)
- added R8: 0402WGF1002TCE, easyeda2kicad:R0402, F.Cu at (62.7, 77.2)
- added R8: 0402WGF1002TCE, easyeda2kicad:R0402, F.Cu at (292.9, 93.2)
- added R9: 0402WGF5101TCE, easyeda2kicad:R0402, F.Cu at (68.5, 44.7)
- added R9: 0402WGF5101TCE, easyeda2kicad:R0402, F.Cu at (279.0, 34.7)
- added REF**: MountingHole_2.2mm_M2, MountingHole:MountingHole_2.2mm_M2, F.Cu at (233.9, 45.9)
- added REF**: MountingHole_2.2mm_M2, MountingHole:MountingHole_2.2mm_M2, F.Cu at (252.5, 99.6)
- added REF**: MountingHole_2.2mm_M2, MountingHole:MountingHole_2.2mm_M2, F.Cu at (92.3, 110.3)
- added REF**: MountingHole_2.2mm_M2, MountingHole:MountingHole_2.2mm_M2, F.Cu at (196.7, 67.4)
- added REF**: MountingHole_2.2mm_M2, MountingHole:MountingHole_2.2mm_M2, F.Cu at (111.0, 56.5)
- added REF**: MountingHole_2.2mm_M2, MountingHole:MountingHole_2.2mm_M2, F.Cu at (148.2, 78.0)
- added S1: Choc HEX, hexcaps:PG1350_hotswap_reversed, F.Cu at (184.3, 45.9)
- added S1: Choc HEX, hexcaps:PG1350_hotswap, B.Cu at (160.6, 56.5)
- added S10: Choc HEX, hexcaps:PG1350_hotswap_reversed, F.Cu at (221.5, 67.4)
- added S10: Choc HEX, hexcaps:PG1350_hotswap, B.Cu at (123.4, 78.0)
- added S11: Choc HEX, hexcaps:PG1350_hotswap_reversed, F.Cu at (258.7, 110.4)
- added S11: Choc HEX, hexcaps:PG1350_hotswap, B.Cu at (86.2, 121.0)
- added S12: Choc HEX, hexcaps:PG1350_hotswap_reversed, F.Cu at (240.1, 35.1)
- added S12: Choc HEX, hexcaps:PG1350_hotswap, B.Cu at (104.8, 45.8)
- added S13: Choc HEX, hexcaps:PG1350_hotswap_reversed, F.Cu at (240.1, 56.6)
- added S13: Choc HEX, hexcaps:PG1350_hotswap, B.Cu at (104.8, 67.3)
- added S14: Choc HEX, hexcaps:PG1350_hotswap_reversed, F.Cu at (240.1, 78.1)
- added S14: Choc HEX, hexcaps:PG1350_hotswap, B.Cu at (104.8, 88.8)
- added S15: Choc HEX, hexcaps:PG1350_hotswap_reversed, F.Cu at (277.4, 99.6)
- added S15: Choc HEX, hexcaps:PG1350_hotswap, B.Cu at (67.5, 110.3)
- added S16: Choc HEX, hexcaps:PG1350_hotswap_reversed, F.Cu at (258.7, 45.9)
- added S16: Choc HEX, hexcaps:PG1350_hotswap, B.Cu at (86.2, 56.5)
- added S17: Choc HEX, hexcaps:PG1350_hotswap_reversed, F.Cu at (258.7, 67.4)
- added S17: Choc HEX, hexcaps:PG1350_hotswap, B.Cu at (86.2, 78.0)
- added S18: Choc HEX, hexcaps:PG1350_hotswap_reversed, F.Cu at (258.7, 88.9)
- added S18: Choc HEX, hexcaps:PG1350_hotswap, B.Cu at (86.2, 99.5)
- added S19: Choc HEX, hexcaps:PG1350_hotswap_reversed, F.Cu at (296.0, 110.4)
- added S19: Choc HEX, hexcaps:PG1350_hotswap, B.Cu at (48.9, 121.0)
- added S2: Choc HEX, hexcaps:PG1350_hotswap_reversed, F.Cu at (184.3, 67.4)
- added S2: Choc HEX, hexcaps:PG1350_hotswap, B.Cu at (160.6, 78.0)
- added S20: Choc HEX, hexcaps:PG1350_hotswap_reversed, F.Cu at (296.0, 45.9)
- added S20: Choc HEX, hexcaps:PG1350_hotswap, B.Cu at (48.9, 56.5)
- added S3: Choc HEX, hexcaps:PG1350_hotswap_reversed, F.Cu at (184.3, 88.9)
- added S3: Choc HEX, hexcaps:PG1350_hotswap, B.Cu at (160.6, 99.5)
- added S4: Choc HEX, hexcaps:PG1350_hotswap_reversed, F.Cu at (202.9, 35.1)
- added S4: Choc HEX, hexcaps:PG1350_hotswap, B.Cu at (142.0, 45.8)
- added S5: Choc HEX, hexcaps:PG1350_hotswap_reversed, F.Cu at (202.9, 56.6)
- added S5: Choc HEX, hexcaps:PG1350_hotswap, B.Cu at (142.0, 67.3)
- added S6: Choc HEX, hexcaps:PG1350_hotswap_reversed, F.Cu at (202.9, 78.1)
- added S6: Choc HEX, hexcaps:PG1350_hotswap, B.Cu at (142.0, 88.8)
- added S7: Choc HEX, hexcaps:PG1350_hotswap_reversed, F.Cu at (240.1, 99.6)
- added S7: Choc HEX, hexcaps:PG1350_hotswap, B.Cu at (104.8, 110.3)
- added S8: Choc HEX, hexcaps:PG1350_hotswap_reversed, F.Cu at (221.5, 24.4)
- added S8: Choc HEX, hexcaps:PG1350_hotswap, B.Cu at (123.4, 35.0)
- added S9: Choc HEX, hexcaps:PG1350_hotswap_reversed, F.Cu at (221.5, 45.9)
- added S9: Choc HEX, hexcaps:PG1350_hotswap, B.Cu at (123.4, 56.5)
- added SW1: TS-1088-AR02016, easyeda2kicad:SW-SMD_L3.9-W3.0-P4.45, F.Cu at (63.4, 79.4)
- added SW1: TS-1088-AR02016, easyeda2kicad:SW-SMD_L3.9-W3.0-P4.45, F.Cu at (294.0, 91.0)
- added U1: SN74LVC1G17DBVR, easyeda2kicad:SOT-23-5_L3.0-W1.7-P0.95-LS2.8-BR, F.Cu at (278.1, 56.8)
- added U1: SN74LVC1G17DBVR, easyeda2kicad:SOT-23-5_L3.0-W1.7-P0.95-LS2.8-BR, F.Cu at (69.8, 67.5)
- added U2: E73-2G4M08S1C, easyeda2kicad:WIRELM-SMD_E73-2G4M08S1C, F.Cu at (53.5, 88.8)
- added U2: E73-2G4M08S1C, easyeda2kicad:WIRELM-SMD_E73-2G4M08S1C, F.Cu at (291.4, 78.1)
- added U4: S2B-PH-K-S(LF)(SN), easyeda2kicad:CONN-TH_S2B-PH-K-S-LF-SN, B.Cu at (61.6, 47.4)
- added U4: S2B-PH-K-S(LF)(SN), easyeda2kicad:CONN-TH_S2B-PH-K-S-LF-SN, B.Cu at (272.0, 35.9)
- added U5: BL8573CS8TR, easyeda2kicad:ESOP-8_L4.9-W3.9-P1.27-LS6.0-BL-EP, F.Cu at (277.0, 40.5)
- added U5: BL8573CS8TR, easyeda2kicad:ESOP-8_L4.9-W3.9-P1.27-LS6.0-BL-EP, F.Cu at (67.5, 50.9)
- added U6: DW01A_C42380662, easyeda2kicad:SOT-23-6_L2.9-W1.6-P0.95-LS2.9-BL, F.Cu at (276.2, 45.5)
- added U6: DW01A_C42380662, easyeda2kicad:SOT-23-6_L2.9-W1.6-P0.95-LS2.9-BL, F.Cu at (64.6, 56.4)
- added U7: LP5024RSMR, easyeda2kicad:VQFN-32_L4.0-W4.0-P0.40-TL-EP, F.Cu at (71.3, 87.6)
- added U7: LP5024RSMR, easyeda2kicad:VQFN-32_L4.0-W4.0-P0.40-TL-EP, F.Cu at (273.7, 78.3)
- added U8: MAX17048, PCM_SparkFun-Semiconductor-Standard:DFN-8_2x2mm_P0.5mm_EP1.2x0.8mm, F.Cu at (62.4, 66.7)
- added U8: MAX17048, PCM_SparkFun-Semiconductor-Standard:DFN-8_2x2mm_P0.5mm_EP1.2x0.8mm, F.Cu at (280.1, 66.3)
- added U9: USBLC6-2SC6, Package_TO_SOT_SMD:SOT-23-6, F.Cu at (285.1, 32.0)
- added U9: USBLC6-2SC6, Package_TO_SOT_SMD:SOT-23-6, F.Cu at (59.4, 63.3)
- added USBC1: TYPE-C-31-M-12, easyeda2kicad:USB-C_SMD-TYPE-C-31-M-12_1, F.Cu at (277.4, 28.7)
- added USBC1: TYPE-C-31-M-12, easyeda2kicad:USB-C_SMD-TYPE-C-31-M-12_1, F.Cu at (67.5, 39.4)
- added VBUS: TestPoint_THTPad_D2.0mm_Drill1.0mm, TestPoint:TestPoint_THTPad_D2.0mm_Drill1.0mm, F.Cu at (286.5, 37.0)
- added VBUS: TestPoint_THTPad_D2.0mm_Drill1.0mm, TestPoint:TestPoint_THTPad_D2.0mm_Drill1.0mm, F.Cu at (73.3, 46.0)
- added VDD_nrf: TestPoint_THTPad_D2.0mm_Drill1.0mm, TestPoint:TestPoint_THTPad_D2.0mm_Drill1.0mm, F.Cu at (278.6, 61.9)
- added VDD_nrf: TestPoint_THTPad_D2.0mm_Drill1.0mm, TestPoint:TestPoint_THTPad_D2.0mm_Drill1.0mm, F.Cu at (67.2, 75.5)
- added X1: FC-13532.768KHZ9PF20PPM, easyeda2kicad:OSC-SMD_L3.2-W1.5, F.Cu at (62.8, 92.9)
- added X1: FC-13532.768KHZ9PF20PPM, easyeda2kicad:OSC-SMD_L3.2-W1.5, F.Cu at (282.1, 74.3)
- moved C10 18.7 mm to (62.8, 64.4), turned to 0 degrees
- moved R19 7.56 mm to (67.9, 62.9)
- moved U10 7.25 mm to (69.4, 62.8)
- moved C13 4.92 mm to (66.2, 62.4), turned to 0 degrees
- moved R15 1.17 mm to (62.2, 51.6)
- moved R18 1.17 mm to (62.2, 50.4)
Routing:
- net /PWR: track 1238.7 -> 1298.0 mm, vias 45 -> 50
- net /ROW3: track 281.1 -> 255.3 mm, vias 12 -> 6
- net GND: track 26.9 -> 7.27 mm, vias 481 -> 1173
- net /COL2: track 493.9 -> 513.1 mm
- net /SDA: track 56.1 -> 75.0 mm, vias 4 -> 5
- net /VBUS_RAW: track 56.5 -> 38.2 mm, vias 12 -> 6
- net /D-: track 151.0 -> 134.0 mm, vias 10 -> 8
- net /D+: track 147.4 -> 131.3 mm, vias 10 -> 8
- net /PWR_BTN: track 63.1 -> 77.0 mm, vias 3 -> 4
- net /VDD_nRF: track 152.2 -> 165.8 mm, vias 8 -> 7
- net /SCL: track 50.2 -> 63.2 mm
- net /ROW2: track 255.9 -> 267.6 mm
- net /COL4: track 361.6 -> 372.5 mm
- net /ROW4: track 196.8 -> 207.0 mm, vias 3 -> 2
- net Net-(D8-Pad1): track 23.5 -> 13.6 mm
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Other:
- outline, holes or cut-outs redrawn
