File: kicad/right.kicad_sch (KiCad schematic)
At the start: 102 parts, among them Q1 PMF170XP,115, Q2 FS8205A_C2830320, SW1 TS-1088-AR02016, U1 SN74LVC1G17DBVR, U10 SN74LVC1G74DQER, U2 E73-2G4M08S1C, U4 S2B-PH-K-S(LF)(SN), U5 BL8573CS8TR, U6 DW01A_C42380662, U7 LP5024RSMR, U8 MAX17048, U9 USBLC6-2SC6, X1 FC-13532.768KHZ9PF20PPM

Commit message: rewired and finalized right side. updated panel. changed dnp of some components on both sides
Parts:
- C1, C3: value 0402CG120F500NT -> 0402CG120J500NT; LCSC Part C182477 -> C1547
- U9: LCSC Part (none) -> C7519; LSCS Part C7519 -> (none)
Connections:
- net LED17: now also U7.16 (OUT15); no longer U7.15 (OUT14)
- net LED20: now also U7.24 (OUT23); no longer U7.22 (OUT21)
- net LED3: now also U7.9 (OUT8); no longer U7.10 (OUT9)
- net VBUS: now also U9.5 (VBUS)
- net VBUS_RAW: no longer U9.5 (VBUS)
- no-connect marks 21 -> 22
Changed lines of the file:
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@@
 	)
 	(no_connect
-		(at 134.62 49.53)
-	)
-	(no_connect
 		(at 280.67 33.02)
 	)
@@
 	)
 	(no_connect
+		(at 134.62 64.77)
+	)
+	(no_connect
 		(at 313.69 71.12)
 	)
@@
 	)
 	(no_connect
-		(at 134.62 44.45)
-	)
-	(no_connect
 		(at 340.36 29.21)
 	)
@@
 	)
 	(no_connect
+		(at 160.02 54.61)
+	)
+	(no_connect
+		(at 160.02 52.07)
+	)
+	(no_connect
 		(at 280.67 35.56)
 	)
@@
 	)
 	(no_connect
-		(at 134.62 46.99)
+		(at 134.62 52.07)
 	)
 	(no_connect
@@
 	)
 	(bus_entry
+		(at 128.27 67.31)
+		(size -2.54 2.54)
+		(stroke
+			(width 0)
+			(type default)
+		)
+	)
+	(bus_entry
 		(at 118.11 55.88)
 		(size 2.54 -2.54)
@@
 	)
 	(bus_entry
-		(at 128.27 64.77)
-		(size -2.54 2.54)
-		(stroke
-			(width 0)
-			(type default)
-		)
-	)
-	(bus_entry
 		(at 128.27 34.29)
 		(size -2.54 2.54)
@@
 	)
 	(bus_entry
-		(at 128.27 52.07)
-		(size -2.54 2.54)
-		(stroke
-			(width 0)
-			(type default)
-		)
-	)
-	(bus_entry
 		(at 118.11 50.8)
 		(size 2.54 -2.54)
@@
 	)
 	(bus_entry
-		(at 166.37 54.61)
+		(at 166.37 49.53)
 		(size 2.54 2.54)
 		(stroke
@@
 	)
 	(bus_entry
+		(at 128.27 49.53)
+		(size -2.54 2.54)
+		(stroke
+			(width 0)
+			(type default)
+		)
+	)
+	(bus_entry
 		(at 118.11 40.64)
 		(size 2.54 -2.54)
@@
 	(wire
 		(pts
-			(xy 128.27 64.77) (xy 134.62 64.77)
-		)
-		(stroke
-			(width 0)
-			(type default)
-		)
-	)
-	(wire
-		(pts
 			(xy 280.67 179.07) (xy 280.67 181.61)
 		)
@@
 	(wire
 		(pts
-			(xy 160.02 54.61) (xy 166.37 54.61)
-		)
-		(stroke
-			(width 0)
-			(type default)
-		)
-	)
-	(wire
-		(pts
 			(xy 91.44 90.17) (xy 91.44 63.5)
 		)
@@
 	(wire
 		(pts
+			(xy 160.02 49.53) (xy 166.37 49.53)
+		)
+		(stroke
+			(width 0)
+			(type default)
+		)
+	)
+	(wire
+		(pts
 			(xy 351.79 231.14) (xy 351.79 233.68)
 		)
@@
 	(wire
 		(pts
+			(xy 128.27 67.31) (xy 134.62 67.31)
+		)
+		(stroke
+			(width 0)
+			(type default)
+		)
+	)
+	(wire
+		(pts
 			(xy 78.74 64.77) (xy 78.74 77.47)
 		)
@@
 	(wire
 		(pts
-			(xy 280.67 204.47) (xy 280.67 209.55)
-		)
-		(stroke
-			(width 0)
-			(type default)
-		)
-	)
-	(wire
-		(pts
 			(xy 78.74 77.47) (xy 78.74 90.17)
 		)
@@
 	(wire
 		(pts
+			(xy 128.27 49.53) (xy 134.62 49.53)
+		)
+		(stroke
+			(width 0)
+			(type default)
+		)
+	)
+	(wire
+		(pts
 			(xy 104.14 68.58) (xy 118.11 68.58)
 		)
@@
 	(wire
 		(pts
-			(xy 128.27 52.07) (xy 134.62 52.07)
-		)
-		(stroke
-			(width 0)
-			(type default)
-		)
-	)
-	(wire
-		(pts
 			(xy 199.39 224.79) (xy 195.58 224.79)
 		)
@@
 		)
 	)
+	(label "VBUS"
+		(at 280.67 209.55 180)
+		(effects
+			(font
+				(size 1.27 1.27)
+			)
+			(justify right bottom)
+		)
+	)
 	(label "BAT+"
 		(at 335.28 152.4 180)
@@
 		)
 	)
+	(label "LED20"
+		(at 160.02 49.53 0)
+		(effects
+			(font
+				(size 1.27 1.27)
+			)
+			(justify left bottom)
+		)
+	)
 	(label "SCL"
 		(at 306.07 71.12 270)
@@
 		)
 	)
-	(label "LED3"
-		(at 134.62 52.07 180)
-		(effects
-			(font
-				(size 1.27 1.27)
-			)
-			(justify right bottom)
-		)
-	)
-	(label "LED20"
-		(at 160.02 54.61 0)
-		(effects
-			(font
-				(size 1.27 1.27)
-			)
-			(justify left bottom)
-		)
-	)
 	(label "D+"
 		(at 285.75 214.63 0)
@@
 		)
 	)
+	(label "LED3"
+		(at 134.62 49.53 180)
+		(effects
+			(font
+				(size 1.27 1.27)
+			)
+			(justify right bottom)
+		)
+	)
 	(label "VDD_nRF"
 		(at 311.15 71.12 270)
@@
 		)
 	)
+	(label "LED17"
+		(at 134.62 67.31 180)
+		(effects
+			(font
+				(size 1.27 1.27)
+			)
+			(justify right bottom)
+		)
+	)
 	(label "LED8"
 		(at 118.11 45.72 180)
@@
 		)
 	)
-	(label "LED17"
-		(at 134.62 64.77 180)
-		(effects
-			(font
-				(size 1.27 1.27)
-			)
-			(justify right bottom)
-		)
-	)
 	(label "SCL"
 		(at 213.36 36.83 270)
@@
 			)
 		)
-		(property "Value" "0402CG120F500NT"
+		(property "Value" "0402CG120J500NT"
 			(at 299.72 93.98 0)
 			(hide yes)
@@
 			)
 		)
-		(property "Datasheet" "https://lcsc.com/product-detail/Multilayer-Ceramic-Capacitors-MLCC-SMD-SMT_12pF-120R-1-50V_C182477.html"
+		(property "Datasheet" "https://lcsc.com/datasheet/C1547.pdf"
 			(at 285.75 93.98 0)
 			(hide yes)
@@
 			)
 		)
-		(property "LCSC Part" "C182477"
+		(property "LCSC Part" "C1547"
 			(at 301.752 93.98 0)
 			(show_name no)
@@
 			)
 		)
-		(property "Value" "0402CG120F500NT"
+		(property "Value" "0402CG120J500NT"
 			(at 281.94 93.98 0)
 			(hide yes)
@@
 			)
 		)
-		(property "Datasheet" "https://lcsc.com/product-detail/Multilayer-Ceramic-Capacitors-MLCC-SMD-SMT_12pF-120R-1-50V_C182477.html"
+		(property "Datasheet" "https://lcsc.com/datasheet/C1547.pdf"
 			(at 295.91 93.98 0)
 			(hide yes)
@@
 			)
 		)
-		(property "LCSC Part" "C182477"
+		(property "LCSC Part" "C1547"
 			(at 279.908 93.98 0)
 			(show_name no)
@@
 			)
 		)
-		(property "LSCS Part" "C7519"
+		(property "LCSC Part" "C7519"
 			(at 280.67 214.63 0)
 			(hide yes)
