File: kicad/right.kicad_sch (KiCad schematic)
At the start: 102 parts, among them Q1 PMF170XP,115, Q2 FS8205A_C2830320, SW1 TS-1088-AR02016, U1 SN74LVC1G17DBVR, U10 SN74LVC1G74DQER, U2 E73-2G4M08S1C, U4 S2B-PH-K-S(LF)(SN), U5 BL8573CS8TR, U6 DW01A_C42380662, U7 LP5024RSMR, U8 MAX17048, U9 USBLC6-2SC6, X1 FC-13532.768KHZ9PF20PPM

Commit message: docs: update charger protection and bring-up checklist
- document selectable 96.5 kΩ and 102 kΩ charge-current settings
- add USB-C TVS and 1.5 A polyfuse protection details
- update IP2312U charger and DW01A protection wiring
- mark completed schematic and ERC checklist items
- revise PCB placement, routing, BOM, and bring-up procedures
Parts:
- removed R11: RC0402FR-07680RL, easyeda2kicad:R0402, symbol easyeda2kicad:RC0201FR-07680RL
- removed R15, R18: 0402WGF1002TCE, easyeda2kicad:R0402, symbol easyeda2kicad:RC0402FR-0710KL
- removed U5: BL8573CS8TR, easyeda2kicad:ESOP-8_L4.9-W3.9-P1.27-LS6.0-BL-EP, symbol easyeda2kicad:BL8573CS8TR
- added C11, C12, C15, C2, C4: 22uF, easyeda2kicad:C0805, symbol easyeda2kicad:CL21A226KOQNNNE
- added C14: CL05B104KB54PNC, easyeda2kicad:C0402, symbol easyeda2kicad:GRM033C71C104KE14D
- added JP1: 96.5k, Jumper:SolderJumper-2_P1.3mm_Open_TrianglePad1.0x1.5mm, symbol Jumper:SolderJumper_2_Open
- added JP2: 102k, Jumper:SolderJumper-2_P1.3mm_Open_TrianglePad1.0x1.5mm, symbol Jumper:SolderJumper_2_Open
- added L2: (no value), Library:BCIHP0420SC-1R0M, symbol Library:BCIHP0420SC-1R0M
- added R12, R15, R18: 0.5Ω, easyeda2kicad:R0402, symbol easyeda2kicad:0402WGF500LTCE
- added R20, R21, R24, R25: 1k, easyeda2kicad:R0402, symbol easyeda2kicad:0402WGF1001TCE
- added R22, R23, R3: 102k, easyeda2kicad:R0402, symbol easyeda2kicad:RT0402BRD07102KL
- added R4: 96.5k, easyeda2kicad:R0402, symbol easyeda2kicad:RT0402BRD07102KL
- added U11: SMF5.0A, easyeda2kicad:SOD-123FL_L2.8-W1.8-LS3.6-RD, symbol easyeda2kicad:SMF5.0A_C2990427
- added U3: IP2312, easyeda2kicad:SOP-8_L4.9-W3.9-P1.27-LS6.0-BL-EP, symbol easyeda2kicad:IP2312
Connections:
- net BAT+: now also C12.2, L2.2, R18.1, R20.1, R21.2, R25.1; no longer U6.5 (VDD)
- net GND: now also C11.1, C12.1, C15.1, C2.1, C4.1, R22.1, R23.1, R24.1, R3.2, R4.2, U11.2, U3.9 (EP); no longer Q2.3 (S2), U4.2, U6.6 (VSS)
- net VBUS: now also C15.2, C2.2, R12.1, U3.8 (VIN)
- net VBUS_RAW: now also U11.1
- net CHRG: no longer names the net of U2.41 (NF1)
- net STDBY: no longer names the net of U2.43 (NF2)
- new net: C14.1, R21.1, U6.5 (VDD)
- new net: C4.2, R15.2
- new net: R22.2, R23.2, U3.4 (NTC)
- new net: R12.2, R15.1
- new net: JP1.2 (B), R4.1
- new net: R24.2, U6.2 (VM)
- new net: JP2.2 (B), R3.1
- new net: C11.2, R18.2, U3.5 (BAT)
- new net: R20.2, U3.2 (TEST)
- new net: R25.2, U3.3 (D2)
- new net: L2.1, U3.7 (SW)
- new net BAT-: C14.2, Q2.3 (S2), U4.2, U6.6 (VSS)
- new net ICHG: JP1.1 (A), JP2.1 (A), U3.6 (ICHG)
- now unconnected: Q2.2 (D1/D2), Q2.5 (D1/D2)
- no-connect marks 22 -> 23
Other:
- moved on the sheet: C10, C13, C9, D1, F1, Q1, R10, R13, R19, R5, R7, R9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

Commit message: finished right part. changed inductor for charger, changed resistor for driver, and added some caps.
Parts:
- removed D10, D11, D12, D13, D14, D15, D16, D17, D18, D19, D2, D20, D3, D4, D5, D6, D7, D8, D9: CDSQC4148-HF, :X1-DFN1006-2_L1.0-W0.6-RD, symbol easyeda2kicad:CDSQC4148-HF
- removed L2: (no value), Library:BCIHP0420SC-1R0M, symbol Library:BCIHP0420SC-1R0M
- removed R6: ERA2AED753X, easyeda2kicad:R0402, symbol easyeda2kicad:ERA2AED753X
- added C16: CL05B104KB54PNC, easyeda2kicad:C0402, symbol easyeda2kicad:GRM033C71C104KE14D
- added C17, C18, C19: 22uF, easyeda2kicad:C0805, symbol easyeda2kicad:CL21A226KOQNNNE
- added L2: 1uH, easyeda2kicad:IND-SMD_L2.5-W2.0, symbol easyeda2kicad:TMS252012ALM-1R0MTAA
- added R1: 14k7 1% 0805, easyeda2kicad:R0805, symbol easyeda2kicad:0805W8F1472T5E
- S1, S14, S19, S20: footprint hexcaps:PG1350_hotswap -> hexcaps:PG1350_hotswap_reversed
- S10: renamed from S17; footprint hexcaps:PG1350_hotswap -> hexcaps:PG1350_hotswap_reversed
- S11: renamed from S3; footprint hexcaps:PG1350_hotswap -> hexcaps:PG1350_hotswap_reversed
- S12: renamed from S6; footprint hexcaps:PG1350_hotswap -> hexcaps:PG1350_hotswap_reversed
- S13: renamed from S10; footprint hexcaps:PG1350_hotswap -> hexcaps:PG1350_hotswap_reversed
- S15: renamed from S18; footprint hexcaps:PG1350_hotswap -> hexcaps:PG1350_hotswap_reversed
- S16: renamed from S7; footprint hexcaps:PG1350_hotswap -> hexcaps:PG1350_hotswap_reversed
- S17: renamed from S11; footprint hexcaps:PG1350_hotswap -> hexcaps:PG1350_hotswap_reversed
- S18: renamed from S15; footprint hexcaps:PG1350_hotswap -> hexcaps:PG1350_hotswap_reversed
- S2: renamed from S4; footprint hexcaps:PG1350_hotswap -> hexcaps:PG1350_hotswap_reversed
- S3: renamed from S8; footprint hexcaps:PG1350_hotswap -> hexcaps:PG1350_hotswap_reversed
- S4: renamed from S12; footprint hexcaps:PG1350_hotswap -> hexcaps:PG1350_hotswap_reversed
- S5: renamed from S16; footprint hexcaps:PG1350_hotswap -> hexcaps:PG1350_hotswap_reversed
- S6: renamed from S2; footprint hexcaps:PG1350_hotswap -> hexcaps:PG1350_hotswap_reversed
- S7: renamed from S5; footprint hexcaps:PG1350_hotswap -> hexcaps:PG1350_hotswap_reversed
- S8: renamed from S9; footprint hexcaps:PG1350_hotswap -> hexcaps:PG1350_hotswap_reversed
- S9: renamed from S13; footprint hexcaps:PG1350_hotswap -> hexcaps:PG1350_hotswap_reversed
- renumbered C7 to C1, C11 to C10, C4 to C11, C2 to C12, C10 to C14, C14 to C15, C8 to C2, C5 to C3, C6 to C4, C1 to C5, C3 to C6, C12 to C7, C9 to C8, C15 to C9, JP2 to JP1, JP1 to JP2, LED17 to LED10, LED4 to LED11, LED14 to LED12, LED11 to LED13, LED8 to LED14, LED18 to LED15, LED15 to LED16, LED12 to LED17, LED19 to LED18, LED16 to LED19, LED5 to LED2, LED2 to LED3, LED9 to LED4, LED6 to LED5, LED3 to LED6, LED13 to LED7, LED10 to LED8, LED7 to LED9, R9 to R10, R25 to R11, R18 to R12, R7 to R13, R15 to R14, R23 to R15, R22 to R16, R10 to R17, R19 to R18, R5 to R19, R14 to R2, R3 to R20, R4 to R21, R21 to R22, R13 to R23, R16 to R3, R17 to R4, R1 to R5, R2 to R6, R8 to R7, R20 to R8, R12 to R9, U2 to U1, U6 to U10, U7 to U2, U10 to U4, U1 to U5, U11 to U6, U9 to U7, U4 to U8, U8 to U9
Connections:
- net ROW2 is gone; now on net LED_EN: U1.10 (AI6)
- net BAT+: now also L2.1
- net BAT_ALTR: now also U1.35 (P0.24); no longer U1.18 (AI2)
- net D+: no longer U7.6 (I/O1), USBC1.A6 (DP1), USBC1.B6 (DP2)
- net D-: no longer U7.4 (I/O2), USBC1.A7 (DN1), USBC1.B7 (DN2)
- net GND: now also S1.2, S10.2, S11.2, S12.2, S13.2, S14.2, S15.2, S16.2, S17.2, S18.2, S19.2, S2.2, S3.2, S4.2, S5.2, S6.2, S7.2, S8.2, S9.2, C16.2, C17.1, C18.1, C19.1, R1.2
- net LED1: now also U2.18 (OUT17); no longer U2.17 (OUT16)
- net LED10: now also LED10.1, U2.17 (OUT16); no longer LED8.1, U2.7 (OUT6)
- net LED11: now also LED11.1, U2.12 (OUT11); no longer LED13.1, U2.3 (OUT2)
- net LED12: now also LED12.1, U2.11 (OUT10); no longer LED17.1, U2.20 (OUT19)
- net LED13: now also LED13.1, U2.10 (OUT9); no longer LED7.1, U2.14 (OUT13)
- net LED14: now also LED14.1, U2.9 (OUT8); no longer LED12.1, U2.6 (OUT5)
- net LED15: now also LED15.1, U2.8 (OUT7); no longer LED16.1, U2.2 (OUT1)
- net LED16: now also LED16.1, U2.7 (OUT6); no longer LED19.1, U2.21 (OUT20)
- net LED17: now also LED17.1, U2.6 (OUT5); no longer LED10.1, U2.16 (OUT15)
- net LED18: now also LED18.1; no longer LED15.1
- net LED19: now also LED19.1, U2.4 (OUT3); no longer LED18.1, U2.1 (OUT0)
- net LED2: now also LED2.1, U2.19 (OUT18); no longer LED3.1, U2.11 (OUT10)
- net LED3: now also LED3.1, U2.20 (OUT19); no longer LED6.1, U2.9 (OUT8)
- net LED4: now also LED4.1, U2.21 (OUT20); no longer LED11.1, U2.18 (OUT17)
- net LED5: now also LED5.1, U2.22 (OUT21); no longer LED2.1, U2.12 (OUT11)
- net LED6: now also LED6.1, U2.13 (OUT12); no longer LED5.1, U2.8 (OUT7)
- net LED7: now also LED7.1, U2.14 (OUT13); no longer LED9.1, U2.4 (OUT3)
- net LED8: now also LED8.1, U2.15 (OUT14); no longer LED14.1, U2.19 (OUT18)
- net LED9: now also LED9.1, U2.16 (OUT15); no longer LED4.1, U2.13 (OUT12)
- net LED_EN: no longer U1.15 (AI3)
- net PWR: now also C17.2, C18.2, C19.2
- net PWR_BTN_PRESS: now also U1.7 (AI0); no longer U1.4 (AI4)
- net SCL: now also U1.15 (AI3); no longer U1.17 (P1.09)
- net SDA: now also U1.17 (P1.09); no longer U1.16 (P0.08)
- net VBUS: now also C16.1
- net at U2.31 (IREF): now also R1.1
- net at U3.7 (SW): now also L2.2
- net S19: now reaches U1.1 (P1.11)
- net S19: now also S19.1
- net S12: now reaches U1.14 (P0.06)
- net S12: now also S12.1
- net S18: now reaches U1.2 (P1.10)
- net S18: now also S18.1
- net S9: now reaches U1.20 (P12)
- net S9: now also S9.1
- net S10: now reaches U1.22 (P0.07)
- net S10: now also S10.1
- net S17: now reaches U1.3 (P0.03)
- net S17: now also S17.1
- net S7: now reaches U1.30 (P17)
- net S7: now also S7.1
- net S1: now reaches U1.33 (P0.13)
- net S1: now also S1.1
- net S5: now reaches U1.40 (P1.04)
- net S5: now also S5.1
- net S14: now reaches U1.8 (AI5)
- net S14: now also S14.1
- removed net COL1: S1.1, S11.1, S6.1, U1.38 (P1.02)
- removed net COL2: S12.1, S16.1, S2.1, S7.1, U1.36 (P1.00)
- removed net COL3: S13.1, S17.1, S3.1, S8.1, U1.34 (P0.22)
- removed net COL4: S14.1, S18.1, S4.1, S9.1, U1.32 (P0.20)
- removed net COL5: S10.1, S15.1, S19.1, S5.1, U1.6 (P1.13)
- net ROW1: no longer names the net of U1.28 (P15)
- net ROW3 renamed S13
- net S13: now also S13.1
- net ROW4: no longer names the net of U1.9 (AI7)
- new net S11: S11.1, U1.16 (P0.08)
- new net S15: S15.1, U1.6 (P1.13)
- new net S16: S16.1, U1.4 (AI4)
- new net S2: S2.1, U1.34 (P0.22)
- new net S3: S3.1, U1.36 (P1.00)
- new net S4: S4.1, U1.38 (P1.02)
- new net S6: S6.1, U1.18 (AI2)
- new net S8: S8.1, U1.32 (P0.20)
- new net USB_D+: U7.6 (I/O1), USBC1.A6 (DP1), USBC1.B6 (DP2)
- new net USB_D-: U7.4 (I/O2), USBC1.A7 (DN1), USBC1.B7 (DN2)
- no-connect marks 23 -> 7
Other:
- note added: "1 per led row. At the start of row feed trace"
- moved on the sheet: C10, C7, R12, S1, S10, S11, S12, S13, S14, S15, S16, S17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

Commit message: cleaned right half, added test points, and some datasheets to the project
Parts:
- added TP1: BAT+, TestPoint:TestPoint_Pad_D2.0mm, symbol Connector:TestPoint
- added TP10: PM_GATE, TestPoint:TestPoint_Pad_D2.0mm, symbol Connector:TestPoint
- added TP11: DFF_CLK, TestPoint:TestPoint_Pad_D2.0mm, symbol Connector:TestPoint
- added TP2: BAT-, TestPoint:TestPoint_Pad_D2.0mm, symbol Connector:TestPoint
- added TP3: GND, TestPoint:TestPoint_Pad_D2.0mm, symbol Connector:TestPoint
- added TP4: VBUS, TestPoint:TestPoint_Pad_D2.0mm, symbol Connector:TestPoint
- added TP5: PWR, TestPoint:TestPoint_Pad_D2.0mm, symbol Connector:TestPoint
- added TP6: 3V3, TestPoint:TestPoint_Pad_D2.0mm, symbol Connector:TestPoint
- added TP7: PWR_PRESS, TestPoint:TestPoint_Pad_D2.0mm, symbol Connector:TestPoint
- added TP8: SDA, TestPoint:TestPoint_Pad_D2.0mm, symbol Connector:TestPoint
- added TP9: SCL, TestPoint:TestPoint_Pad_D2.0mm, symbol Connector:TestPoint
Connections:
- net BAT+: now also TP1.1
- net BAT-: now also TP2.1
- net GND: now also TP3.1
- net PMOS_gate: now also TP10.1
- net PWR: now also TP5.1
- net PWR_BTN_PRESS: now also TP7.1
- net SCL: now also TP9.1
- net SDA: now also TP8.1
- net VBUS_RAW: now also TP4.1
- net DFF_CLK: now reaches U4.1 (CLK), U5.4 (Y)
- net DFF_CLK: now also TP11.1
- net SWBCLK renamed SWDCLK
- net VDD_nRF renamed 3V3
- net 3V3: now also TP6.1
Other:
- moved on the sheet: R4
