File: kicad/left.kicad_sch (KiCad schematic)
At the start: 102 parts, among them Q1 PMF170XP,115, Q2 FS8205A_C2830320, SW1 TS-1088-AR02016, U1 SN74LVC1G17DBVR, U2 E73-2G4M08S1C, U3 SN74LVC1G74DQER, U4 S2B-PH-K-S(LF)(SN), U5 BL8573CS8TR, U6 DW01A_C42380662, U7 LP5024RSMR, U8 MAX17048, U9 USBLC6-2SC6, X1 FC-13532.768KHZ9PF20PPM

Commit message: fixed u9 to have pin 5 after polyfuse
Connections:
- net VBUS: now also U9.5 (VBUS)
- net VBUS_RAW: no longer U9.5 (VBUS)
Changed lines of the file:
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@@
-		)
-	)
-	(wire
-		(pts
-			(xy 280.67 204.47) (xy 280.67 209.55)
-		)
-		(stroke
-			(width 0)
-			(type default)
 		)
 	)
@@
 		(effects
 			(font
+				(size 1.27 1.27)
+			)
+			(justify right bottom)
+		)
+	)
+	(label "VBUS"
+		(at 280.67 209.55 180)
+		(effects
+			(font
